File: Interface-PCB/RemoteTransistor.kicad_sch (KiCad schematic)
At the start: 23 parts, among them IC2 TBD62783APG, IC3 TBD62783APG, J14 CONN_05JST, J15 CONN_05JST, U3 CD74HC4067_MUX_BREAKOUT

Commit message: Complete Initial Layout of PCB
- aligned to 5mm grid
- 100x100mm board
- update footprints
- align 2 resistors to 2.54mm spacing
Parts:
- renumbered J14 to J13, J15 to J14, R12 to R11, R13 to R12, R14 to R13, R15 to R14, R16 to R15, R17 to R16, R18 to R17, R19 to R18, R20 to R19, R21 to R20, R22 to R21, R23 to R22, R24 to R23, R25 to R24, R26 to R25, R27 to R26
Changed lines of the file:
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@@
   (title_block
     (title "Interface PCB")
-    (date "2023-01-18")
+    (date "2023-01-20")
     (rev "1")
     (company "Team 48 - Planter")
@@
   (symbol (lib_id "power:+3.3V") (at 200.66 52.07 0) (unit 1)
     (in_bom yes) (on_board yes)
-    (property "Reference" "#PWR038" (id 0) (at 200.66 55.88 0)
+    (property "Reference" "#PWR036" (id 0) (at 200.66 55.88 0)
       (effects (font (size 1.27 1.27)) hide)
     )
@@
   (symbol (lib_id "power:+3.3V") (at 181.61 36.83 0) (unit 1)
     (in_bom yes) (on_board yes)
-    (property "Reference" "#PWR037" (id 0) (at 181.61 40.64 0)
+    (property "Reference" "#PWR035" (id 0) (at 181.61 40.64 0)
       (effects (font (size 1.27 1.27)) hide)
     )
@@
   (symbol (lib_id "AA_Custom_Components:CONN_05JST") (at 81.28 114.3 0) (mirror y) (unit 1)
     (in_bom yes) (on_board yes)
-    (property "Reference" "J14" (id 0) (at 80.01 99.06 0)
+    (property "Reference" "J13" (id 0) (at 80.01 99.06 0)
       (effects (font (size 1.143 1.143)) (justify right))
     )
@@
   (symbol (lib_id "power:+12V") (at 53.34 133.35 0) (unit 1)
     (in_bom yes) (on_board yes)
-    (property "Reference" "#PWR035" (id 0) (at 53.34 137.16 0)
+    (property "Reference" "#PWR033" (id 0) (at 53.34 137.16 0)
       (effects (font (size 1.27 1.27)) hide)
     )
@@
   (symbol (lib_id "power:+12V") (at 53.34 171.45 0) (unit 1)
     (in_bom yes) (on_board yes)
-    (property "Reference" "#PWR036" (id 0) (at 53.34 175.26 0)
+    (property "Reference" "#PWR034" (id 0) (at 53.34 175.26 0)
       (effects (font (size 1.27 1.27)) hide)
     )
@@
   (symbol (lib_id "AA_Custom_Components:CONN_05JST") (at 81.28 152.4 0) (mirror y) (unit 1)
     (in_bom yes) (on_board yes)
-    (property "Reference" "J15" (id 0) (at 80.01 137.16 0)
+    (property "Reference" "J14" (id 0) (at 80.01 137.16 0)
       (effects (font (size 1.143 1.143)) (justify right))
     )
@@
   (symbol (lib_id "AA_Custom_Components:GND") (at 21.59 115.57 0) (unit 1)
     (in_bom yes) (on_board yes)
-    (property "Reference" "#GND028" (id 0) (at 22.86 116.84 0)
+    (property "Reference" "#GND027" (id 0) (at 22.86 116.84 0)
       (effects (font (size 1.143 1.143)) (justify left bottom) hide)
     )
@@
   (symbol (lib_id "AA_Custom_Components:GND") (at 21.59 153.67 0) (unit 1)
     (in_bom yes) (on_board yes)
-    (property "Reference" "#GND029" (id 0) (at 22.86 154.94 0)
+    (property "Reference" "#GND028" (id 0) (at 22.86 154.94 0)
       (effects (font (size 1.143 1.143)) (justify left bottom) hide)
     )
@@
   (symbol (lib_id "power:+12V") (at 21.59 107.95 0) (unit 1)
     (in_bom yes) (on_board yes)
-    (property "Reference" "#PWR033" (id 0) (at 21.59 111.76 0)
+    (property "Reference" "#PWR031" (id 0) (at 21.59 111.76 0)
       (effects (font (size 1.27 1.27)) hide)
     )
@@
   (symbol (lib_id "power:+12V") (at 21.59 146.05 0) (unit 1)
     (in_bom yes) (on_board yes)
-    (property "Reference" "#PWR034" (id 0) (at 21.59 149.86 0)
+    (property "Reference" "#PWR032" (id 0) (at 21.59 149.86 0)
       (effects (font (size 1.27 1.27)) hide)
     )
@@
   (symbol (lib_id "AA_Custom_Components:GND") (at 44.45 121.92 0) (unit 1)
     (in_bom yes) (on_board yes)
-    (property "Reference" "#GND030" (id 0) (at 45.72 123.19 0)
+    (property "Reference" "#GND029" (id 0) (at 45.72 123.19 0)
       (effects (font (size 1.143 1.143)) (justify left bottom) hide)
     )
@@
   (symbol (lib_id "AA_Custom_Components:GND") (at 44.45 160.02 0) (unit 1)
     (in_bom yes) (on_board yes)
-    (property "Reference" "#GND031" (id 0) (at 45.72 161.29 0)
+    (property "Reference" "#GND030" (id 0) (at 45.72 161.29 0)
       (effects (font (size 1.143 1.143)) (justify left bottom) hide)
     )
@@
   (symbol (lib_id "AA_Custom_Components:GND") (at 76.2 162.56 0) (unit 1)
     (in_bom yes) (on_board yes)
-    (property "Reference" "#GND033" (id 0) (at 77.47 163.83 0)
+    (property "Reference" "#GND032" (id 0) (at 77.47 163.83 0)
       (effects (font (size 1.143 1.143)) (justify left bottom) hide)
     )
@@
   (symbol (lib_id "AA_Custom_Components:GND") (at 76.2 124.46 0) (unit 1)
     (in_bom yes) (on_board yes)
-    (property "Reference" "#GND032" (id 0) (at 77.47 125.73 0)
+    (property "Reference" "#GND031" (id 0) (at 77.47 125.73 0)
       (effects (font (size 1.143 1.143)) (justify left bottom) hide)
     )
@@
   (symbol (lib_id "AA_Custom_Components:GND") (at 95.25 77.47 0) (unit 1)
     (in_bom yes) (on_board yes)
-    (property "Reference" "#GND034" (id 0) (at 96.52 78.74 0)
+    (property "Reference" "#GND033" (id 0) (at 96.52 78.74 0)
       (effects (font (size 1.143 1.143)) (justify left bottom) hide)
     )
@@
   (symbol (lib_id "AA_Custom_Components:GND") (at 185.42 54.61 0) (unit 1)
     (in_bom yes) (on_board yes)
-    (property "Reference" "#GND035" (id 0) (at 186.69 55.88 0)
+    (property "Reference" "#GND034" (id 0) (at 186.69 55.88 0)
       (effects (font (size 1.143 1.143)) (justify left bottom) hide)
     )
@@
   (symbol (lib_id "Device:R") (at 72.39 68.58 0) (unit 1)
     (in_bom yes) (on_board yes)
-    (property "Reference" "R16" (id 0) (at 74.168 67.4116 0)
+    (property "Reference" "R15" (id 0) (at 74.168 67.4116 0)
       (effects (font (size 1.27 1.27)) (justify left))
     )
@@
   (symbol (lib_id "Device:R") (at 133.35 68.58 0) (unit 1)
     (in_bom yes) (on_board yes)
-    (property "Reference" "R24" (id 0) (at 135.128 67.4116 0)
+    (property "Reference" "R23" (id 0) (at 135.128 67.4116 0)
       (effects (font (size 1.27 1.27)) (justify left))
     )
@@
   (symbol (lib_id "Device:R") (at 80.01 68.58 0) (unit 1)
     (in_bom yes) (on_board yes)
-    (property "Reference" "R17" (id 0) (at 81.788 67.4116 0)
+    (property "Reference" "R16" (id 0) (at 81.788 67.4116 0)
       (effects (font (size 1.27 1.27)) (justify left))
     )
@@
   (symbol (lib_id "Device:R") (at 140.97 68.58 0) (unit 1)
     (in_bom yes) (on_board yes)
-    (property "Reference" "R25" (id 0) (at 142.748 67.4116 0)
+    (property "Reference" "R24" (id 0) (at 142.748 67.4116 0)
       (effects (font (size 1.27 1.27)) (justify left))
     )
@@
   (symbol (lib_id "Device:R") (at 64.77 68.58 0) (unit 1)
     (in_bom yes) (on_board yes)
-    (property "Reference" "R15" (id 0) (at 66.548 67.4116 0)
+    (property "Reference" "R14" (id 0) (at 66.548 67.4116 0)
       (effects (font (size 1.27 1.27)) (justify left))
     )
@@
   (symbol (lib_id "Device:R") (at 87.63 68.58 0) (unit 1)
     (in_bom yes) (on_board yes)
-    (property "Reference" "R18" (id 0) (at 89.408 67.4116 0)
+    (property "Reference" "R17" (id 0) (at 89.408 67.4116 0)
       (effects (font (size 1.27 1.27)) (justify left))
     )
@@
   (symbol (lib_id "Device:R") (at 49.53 68.58 0) (unit 1)
     (in_bom yes) (on_board yes)
-    (property "Reference" "R13" (id 0) (at 51.308 67.4116 0)
+    (property "Reference" "R12" (id 0) (at 51.308 67.4116 0)
       (effects (font (size 1.27 1.27)) (justify left))
     )
@@
   (symbol (lib_id "Device:R") (at 102.87 68.58 0) (unit 1)
     (in_bom yes) (on_board yes)
-    (property "Reference" "R20" (id 0) (at 104.648 67.4116 0)
+    (property "Reference" "R19" (id 0) (at 104.648 67.4116 0)
       (effects (font (size 1.27 1.27)) (justify left))
     )
@@
   (symbol (lib_id "Device:R") (at 41.91 68.58 0) (unit 1)
     (in_bom yes) (on_board yes)
-    (property "Reference" "R12" (id 0) (at 43.688 67.4116 0)
+    (property "Reference" "R11" (id 0) (at 43.688 67.4116 0)
       (effects (font (size 1.27 1.27)) (justify left))
     )
@@
   (symbol (lib_id "Device:R") (at 156.21 68.58 0) (unit 1)
     (in_bom yes) (on_board yes)
-    (property "Reference" "R27" (id 0) (at 157.988 67.4116 0)
+    (property "Reference" "R26" (id 0) (at 157.988 67.4116 0)
       (effects (font (size 1.27 1.27)) (justify left))
     )
@@
   (symbol (lib_id "Device:R") (at 95.25 68.58 0) (unit 1)
     (in_bom yes) (on_board yes)
-    (property "Reference" "R19" (id 0) (at 97.028 67.4116 0)
+    (property "Reference" "R18" (id 0) (at 97.028 67.4116 0)
       (effects (font (size 1.27 1.27)) (justify left))
     )
@@
   (symbol (lib_id "Device:R") (at 148.59 68.58 0) (unit 1)
     (in_bom yes) (on_board yes)
-    (property "Reference" "R26" (id 0) (at 150.368 67.4116 0)
+    (property "Reference" "R25" (id 0) (at 150.368 67.4116 0)
       (effects (font (size 1.27 1.27)) (justify left))
     )
@@
   (symbol (lib_id "Device:R") (at 57.15 68.58 0) (unit 1)
     (in_bom yes) (on_board yes)
-    (property "Reference" "R14" (id 0) (at 58.928 67.4116 0)
+    (property "Reference" "R13" (id 0) (at 58.928 67.4116 0)
       (effects (font (size 1.27 1.27)) (justify left))
     )
@@
   (symbol (lib_id "Device:R") (at 125.73 68.58 0) (unit 1)
     (in_bom yes) (on_board yes)
-    (property "Reference" "R23" (id 0) (at 127.508 67.4116 0)
+    (property "Reference" "R22" (id 0) (at 127.508 67.4116 0)
       (effects (font (size 1.27 1.27)) (justify left))
     )
@@
   (symbol (lib_id "Device:R") (at 110.49 68.58 0) (unit 1)
     (in_bom yes) (on_board yes)
-    (property "Reference" "R21" (id 0) (at 112.268 67.4116 0)
+    (property "Reference" "R20" (id 0) (at 112.268 67.4116 0)
       (effects (font (size 1.27 1.27)) (justify left))
     )
@@
   (symbol (lib_id "Device:R") (at 118.11 68.58 0) (unit 1)
     (in_bom yes) (on_board yes)
-    (property "Reference" "R22" (id 0) (at 119.888 67.4116 0)
-      (effects (font (size 1.27 1.27)) (justify left))
-    )
+    (property "Reference" "R21" (id 0) (at 119.888 67.4116 0)
+      (effects (font (size 1.27 1.27)) (justify left))
+    )
